Commit message: servo with keyboard and joystick

File: src/myactuator_arm/description/urdf/arm_description.urdf.xacro (robot description, xacro)
@@ -279,39 +279,47 @@
     </collision>
   </link>
-  <!-- Link 5: Lower forearm and hand (yaw rotation) -->
+  <!-- Link 5: Lower forearm (yaw rotation) -->
+  <link name="wrist_link">
+    <inertial>
+      <origin xyz="-2.78156e-05 0.00215422 -0.08" rpy="0 0 0"/>
+      <mass value="0.3"/>
+      <inertia ixx="0.001" ixy="0" ixz="0" iyy="0.001" iyz="0" izz="0.0002"/>
+    </inertial>
+    <visual>
+      <origin xyz="0 -0.09 0.023" rpy="1.5708 -1.5708 0"/>
+      <geometry>
+        <mesh filename="package://myactuator_arm/description/meshes/rotor_x4_p36_36.stl"/>
+      </geometry>
+      <material name="dark_purple"/>
+    </visual>
+    <collision>
+      <origin xyz="0 -0.09 0.023" rpy="1.5708 -1.5708 0"/>
+      <geometry>
+        <mesh filename="package://myactuator_arm/description/meshes/rotor_x4_p36_36.stl"/>
+      </geometry>
+    </collision>
+    <visual>
+      <origin xyz="-6.05561e-05 0.00294052 -0.075703" rpy="0 0 0"/>
+      <geometry>
+        <mesh filename="package://myactuator_arm/description/meshes/l_lower_forearm.stl"/>
+      </geometry>
+      <material name="blue"/>
+    </visual>
+    <collision>
+      <origin xyz="-6.05561e-05 0.00294052 -0.075703" rpy="0 0 0"/>
+      <geometry>
+        <mesh filename="package://myactuator_arm/description/meshes/l_lower_forearm.stl"/>
+      </geometry>
+    </collision>
+  </link>
+  <!-- Link 6: End effector / Hand (roll rotation - 6th DOF) -->
   <link name="end_effector_link">
     <inertial>
-      <origin xyz="-2.78156e-05 0.00215422 -0.147028" rpy="0 0 0"/>
-      <mass value="0.558"/>
-      <inertia ixx="0.00382826" ixy="-3.16312e-08" ixz="2.02243e-07" iyy="0.00375463" iyz="-2.11667e-05" izz="0.000416359"/>
-    </inertial>
-    <visual>
-      <origin xyz="0 -0.09 0.023" rpy="1.5708 -1.5708 0"/>
-      <geometry>
-        <mesh filename="package://myactuator_arm/description/meshes/rotor_x4_p36_36.stl"/>
-      </geometry>
-      <material name="dark_purple"/>
-    </visual>
-    <collision>
-      <origin xyz="0 -0.09 0.023" rpy="1.5708 -1.5708 0"/>
-      <geometry>
-        <mesh filename="package://myactuator_arm/description/meshes/rotor_x4_p36_36.stl"/>
-      </geometry>
-    </collision>
-    <visual>
-      <origin xyz="-6.05561e-05 0.00294052 -0.075703" rpy="0 0 0"/>
-      <geometry>
-        <mesh filename="package://myactuator_arm/description/meshes/l_lower_forearm.stl"/>
-      </geometry>
-      <material name="blue"/>
-    </visual>
-    <collision>
-      <origin xyz="-6.05561e-05 0.00294052 -0.075703" rpy="0 0 0"/>
-      <geometry>
-        <mesh filename="package://myactuator_arm/description/meshes/l_lower_forearm.stl"/>
-      </geometry>
-    </collision>
-    <visual>
-      <origin xyz="0 0 -0.252" rpy="0 0 1.5708"/>
+      <origin xyz="0 0 -0.08" rpy="0 0 0"/>
+      <mass value="0.258"/>
+      <inertia ixx="0.002" ixy="0" ixz="0" iyy="0.002" iyz="0" izz="0.0002"/>
+    </inertial>
+    <visual>
+      <origin xyz="0 0 -0.162" rpy="0 0 1.5708"/>
       <geometry>
         <mesh filename="package://myactuator_arm/description/meshes/hand.stl"/>
@@ -322,12 +330,12 @@
     </visual>
     <collision>
-      <origin xyz="0 0 -0.252" rpy="0 0 1.5708"/>
+      <origin xyz="0 0 -0.162" rpy="0 0 1.5708"/>
       <geometry>
         <mesh filename="package://myactuator_arm/description/meshes/hand.stl"/>
       </geometry>
     </collision>
-    <!-- Gripper fingers collision (using simplified hand collision for now) -->
-    <visual>
-      <origin xyz="0 0 -0.252" rpy="0 0 1.5708"/>
+    <!-- Gripper fingers -->
+    <visual>
+      <origin xyz="0 0 -0.162" rpy="0 0 1.5708"/>
       <geometry>
         <mesh filename="package://myactuator_arm/description/meshes/f1.stl"/>
@@ -336,5 +344,5 @@
     </visual>
     <collision>
-      <origin xyz="0 0 -0.252" rpy="0 0 1.5708"/>
+      <origin xyz="0 0 -0.162" rpy="0 0 1.5708"/>
       <geometry>
         <mesh filename="package://myactuator_arm/description/meshes/f1.stl"/>
@@ -342,5 +350,5 @@
     </collision>
     <visual>
-      <origin xyz="0 0 -0.252" rpy="0 0 1.5708"/>
+      <origin xyz="0 0 -0.162" rpy="0 0 1.5708"/>
       <geometry>
         <mesh filename="package://myactuator_arm/description/meshes/f2.stl"/>
@@ -349,5 +357,5 @@
     </visual>
     <collision>
-      <origin xyz="0 0 -0.252" rpy="0 0 1.5708"/>
+      <origin xyz="0 0 -0.162" rpy="0 0 1.5708"/>
       <geometry>
         <mesh filename="package://myactuator_arm/description/meshes/f2.stl"/>
@@ -355,5 +363,5 @@
     </collision>
     <visual>
-      <origin xyz="0 0 -0.252" rpy="0 0 1.5708"/>
+      <origin xyz="0 0 -0.162" rpy="0 0 1.5708"/>
       <geometry>
         <mesh filename="package://myactuator_arm/description/meshes/f3.stl"/>
@@ -362,5 +370,5 @@
     </visual>
     <collision>
-      <origin xyz="0 0 -0.252" rpy="0 0 1.5708"/>
+      <origin xyz="0 0 -0.162" rpy="0 0 1.5708"/>
       <geometry>
         <mesh filename="package://myactuator_arm/description/meshes/f3.stl"/>
@@ -368,5 +376,5 @@
     </collision>
     <visual>
-      <origin xyz="0 0 -0.252" rpy="0 0 1.5708"/>
+      <origin xyz="0 0 -0.162" rpy="0 0 1.5708"/>
       <geometry>
         <mesh filename="package://myactuator_arm/description/meshes/f4.stl"/>
@@ -375,5 +383,5 @@
     </visual>
     <collision>
-      <origin xyz="0 0 -0.252" rpy="0 0 1.5708"/>
+      <origin xyz="0 0 -0.162" rpy="0 0 1.5708"/>
       <geometry>
         <mesh filename="package://myactuator_arm/description/meshes/f4.stl"/>
@@ -381,5 +389,5 @@
     </collision>
     <visual>
-      <origin xyz="0 0 -0.252" rpy="0 0 1.5708"/>
+      <origin xyz="0 0 -0.162" rpy="0 0 1.5708"/>
       <geometry>
         <mesh filename="package://myactuator_arm/description/meshes/f5.stl"/>
@@ -388,5 +396,5 @@
     </visual>
     <collision>
-      <origin xyz="0 0 -0.252" rpy="0 0 1.5708"/>
+      <origin xyz="0 0 -0.162" rpy="0 0 1.5708"/>
       <geometry>
         <mesh filename="package://myactuator_arm/description/meshes/f5.stl"/>
@@ -426,11 +434,20 @@
     <limit lower="-1.57087" upper="1.57072" velocity="16.0" effort="10.0"/>
   </joint>
-  <!-- Joint 5: Elbow yaw -->
+  <!-- Joint 5: Wrist pitch -->
   <joint name="joint5" type="revolute">
     <origin xyz="0 -0.151 0.023" rpy="-1.5708 -1.5708 0"/>
     <parent link="upper_forearm_link"/>
-    <child link="end_effector_link"/>
+    <child link="wrist_link"/>
     <axis xyz="0 0 1"/>
     <limit lower="-1.5708" upper="1.5708" velocity="16.0" effort="10.0"/>
   </joint>
+  <!-- Joint 6: Wrist roll (6th DOF for full Cartesian control) -->
+  <!-- Using Y axis to ensure independence from joint5 (which uses Z after its rpy transform) -->
+  <joint name="joint6" type="revolute">
+    <origin xyz="0 0 -0.09" rpy="0 0 0"/>
+    <parent link="wrist_link"/>
+    <child link="end_effector_link"/>
+    <axis xyz="0 1 0"/>
+    <limit lower="-3.14159" upper="3.14159" velocity="16.0" effort="10.0"/>
+  </joint>
 </robot>

File: src/myactuator_arm_moveit_config/config/myactuator_arm.ros2_control.xacro (robot description, xacro)
@@ -8,36 +8,43 @@
                 <plugin>mock_components/GenericSystem</plugin>
             </hardware>
-            <joint name="joint1">
+            <joint name="shoulder_pitch_joint">
                 <command_interface name="position"/>
                 <state_interface name="position">
-                  <param name="initial_value">${initial_positions['joint1']}</param>
+                  <param name="initial_value">${initial_positions['shoulder_pitch_joint']}</param>
                 </state_interface>
                 <state_interface name="velocity"/>
             </joint>
-            <joint name="joint2">
+            <joint name="shoulder_roll_joint">
                 <command_interface name="position"/>
                 <state_interface name="position">
-                  <param name="initial_value">${initial_positions['joint2']}</param>
+                  <param name="initial_value">${initial_positions['shoulder_roll_joint']}</param>
                 </state_interface>
                 <state_interface name="velocity"/>
             </joint>
-            <joint name="joint3">
+            <joint name="shoulder_yaw_joint">
                 <command_interface name="position"/>
                 <state_interface name="position">
-                  <param name="initial_value">${initial_positions['joint3']}</param>
+                  <param name="initial_value">${initial_positions['shoulder_yaw_joint']}</param>
                 </state_interface>
                 <state_interface name="velocity"/>
             </joint>
-            <joint name="joint4">
+            <joint name="elbow_pitch_joint">
                 <command_interface name="position"/>
                 <state_interface name="position">
-                  <param name="initial_value">${initial_positions['joint4']}</param>
+                  <param name="initial_value">${initial_positions['elbow_pitch_joint']}</param>
                 </state_interface>
                 <state_interface name="velocity"/>
             </joint>
-            <joint name="joint5">
+            <joint name="elbow_yaw_joint">
                 <command_interface name="position"/>
                 <state_interface name="position">
-                  <param name="initial_value">${initial_positions['joint5']}</param>
+                  <param name="initial_value">${initial_positions['elbow_yaw_joint']}</param>
+                </state_interface>
+                <state_interface name="velocity"/>
+            </joint>
+            <joint name="wrist_roll_joint">
+                <command_interface name="position"/>
+                <state_interface name="position">
+                  <param name="initial_value">${initial_positions['wrist_roll_joint']}</param>
                 </state_interface>
                 <state_interface name="velocity"/>

File: src/myactuator_arm_moveit_config/config/myactuator_arm.urdf.xacro (robot description, xacro)
@@ -1,9 +1,6 @@
 <?xml version="1.0"?>
 <robot xmlns:xacro="http://www.ros.org/wiki/xacro" name="myactuator_arm">
-    <xacro:arg name="initial_positions_file" default="initial_positions.yaml" />
-    <!-- Import myactuator_arm urdf file -->
-    <xacro:include filename="$(find myactuator_arm)/description/urdf/arm_full.urdf.xacro" />
-    <!-- Import control_xacro -->
-    <xacro:include filename="myactuator_arm.ros2_control.xacro" />
-    <xacro:myactuator_arm_ros2_control name="FakeSystem" initial_positions_file="$(arg initial_positions_file)"/>
+    <xacro:arg name="initial_positions_file" default="$(find myactuator_arm_moveit_config)/config/initial_positions.yaml" />
+    <!-- Import new 6-DOF robot with ros2_control -->
+    <xacro:include filename="$(find myactuator_arm)/robot_arm_6dof/robot_with_control.urdf.xacro" />
 </robot>
